Commit message: Initial commit: SLAM ready version of four_wheel_2d

File: urdf/four_wheel_2d.urdf.xacro (robot description, xacro)
@@ -1,5 +1,5 @@
 <?xml version="1.0"?>
 <!-- http://wiki.ros.org/urdf/XML/link  -->
-<robot xmlns:xacro="http://www.ros.org/wiki/xacro" name="four_wheels">
+<robot xmlns:xacro="http://www.ros.org/wiki/xacro" name="four_wheel_2d">
     <!-- Define constants -->
     <xacro:property name="pi" value="1.570795"/>
@@ -15,7 +15,7 @@
     <xacro:property name="laser_mass" value="0.1"/>
     <xacro:property name="laser_radius" value="0.05"/>
-    <xacro:property name="laser_length" value="0.04"/>
+    <xacro:property name="laser_length" value="0.05"/>
     <xacro:property name="laser_distance_z" value="${base_height/2 + laser_length/2}"/>
-    <xacro:property name="laser_distance_x" value="0"/>
+    <xacro:property name="laser_distance_x" value="-0.1"/>
     <xacro:property name="camera_size_x" value="0.02"/>
     <xacro:property name="camera_size_y" value="0.1"/>
@@ -24,7 +24,13 @@
     <xacro:property name="camera_distance_y" value="0"/>
     <xacro:property name="camera_distance_z" value="0"/>
+    <xacro:property name="imu_size_x" value="0.05"/>
+    <xacro:property name="imu_size_y" value="0.05"/>
+    <xacro:property name="imu_size_z" value="0.05"/>
+    <xacro:property name="imu_distance_x" value="0.1"/>
+    <xacro:property name="imu_distance_y" value="0"/>
+    <xacro:property name="imu_distance_z" value="${base_height/2 + imu_size_z/2}"/>
     <!-- Include the common gazebo macros -->
-    <xacro:include filename="$(find four_wheel)/urdf/common_gazebo.xacro" />
-    <xacro:include filename="$(find four_wheel)/urdf/inertial_macro.xacro" />
+    <xacro:include filename="$(find four_wheel_2d)/urdf/common_gazebo.xacro" />
+    <xacro:include filename="$(find four_wheel_2d)/urdf/inertial_macro.xacro" />
     <!-- This is the base of the robot -->
     <link name="base_footprint"/>
@@ -91,8 +97,11 @@
     <xacro:wheel name="front_left" x="${base_length * 0.3}" y="${base_width/2 + wheel_length/2}" z="${base_wheel_distance - base_height/2}"/>
     <!-- Include the skid steering drive plugin -->
-    <xacro:include filename="$(find four_wheel)/urdf/four_wheel_drive_gazebo.xacro" />
+    <xacro:include filename="$(find four_wheel_2d)/urdf/four_wheel_drive_gazebo.xacro" />
     <!-- Include the lidar -->
-    <xacro:include filename="$(find four_wheel)/urdf/lidar3d.xacro" />
+    <xacro:include filename="$(find four_wheel_2d)/urdf/lidar2d.xacro" />
     <!-- Include the camera -->
-    <xacro:include filename="$(find four_wheel)/urdf/camera.xacro" />
+    <xacro:include filename="$(find four_wheel_2d)/urdf/camera.xacro" />
+    <!-- Include the IMU -->
+    <xacro:include filename="$(find four_wheel_2d)/urdf/bno055_imu.xacro" />
+    <xacro:add_bno055_imu parent_link="body_link"/>
 </robot>

File: urdf/lidar2d.xacro (robot description, xacro)
@@ -1,10 +1,10 @@
 <?xml version="1.0"?>
 <robot xmlns:xacro="http://www.ros.org/wiki/xacro" >
-    <joint name="velodyne_joint" type="fixed">
+    <joint name="lidar_joint" type="fixed">
         <parent link="body_link"/>
-        <child link="velodyne_link"/>
+        <child link="lidar_link"/>
         <origin xyz="${laser_distance_x} 0 ${laser_distance_z}" rpy="0 0 0"/>
     </joint>
-    <link name="velodyne_link">
+    <link name="lidar_link">
         <visual>
             <geometry>
@@ -22,5 +22,5 @@
         </xacro:inertial_cylinder>
     </link>
-    <gazebo reference="velodyne_link">
+    <gazebo reference="lidar_link">
         <material>Gazebo/Red</material>
         <sensor name="laser" type="ray">
@@ -35,9 +35,4 @@
                         <max_angle>6.28</max_angle>
                     </horizontal>
-                    <vertical>
-                        <samples>16</samples>
-                        <min_angle>-0.2618</min_angle>
-                        <max_angle>0.2618</max_angle>
-                    </vertical>
                 </scan>
                 <range>
@@ -46,10 +41,10 @@
                 </range>
             </ray>
-            <plugin name="gazebo_ros_laser" filename="libgazebo_ros_ray_sensor.so">
+            <plugin name="laser_controller" filename="libgazebo_ros_ray_sensor.so">
                 <ros>
-                <argument>~/out:=velodyne_points</argument>
+                    <argument>~/out:=scan</argument>
                 </ros>
-                <topicName>/velodyne_points</topicName>
-                <frameName>velodyne_link</frameName>
+                <output_type>sensor_msgs/LaserScan</output_type>
+                <frameName>lidar_link</frameName>
             </plugin>
         </sensor>
